File: MAPS-010143/MAPS-010143.kicad_pcb (KiCad board)
At the start: 4 copper layers, 49.2 x 82.9 mm, 85 parts, among them IC1 LM2776DBVT, IC11 MAPS-010144-TR0500, IC2 PE4302-51, IC3 BGB_741L7ESD_E6327, IC4 BGB_741L7ESD_E6327, IC6 PE4302-51, IC7 SN74HC595NSR, IC8 SN74HC595NSR, IC9 MAPS-010144-TR0500, J13 Conn_01x02_Pin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

Commit message: v2 発注記念。
Parts:
- removed U4: TPS7A2033PDQNR, footprints:DQN0004A-MFG
- added IC5: TPS7A2033PDBVR, SamacSys_Parts:SOT95P280X145-5N, B.Cu at (119.2, 70.2)
- moved C9 3.41 mm to (117.6, 67.5)
- moved C21 1.90 mm to (117.5, 74.5)
- moved C10 1.63 mm to (117.7, 73.0)
- moved TP3 0.07 mm to (142.9, 88.6)
- moved TP2 0.05 mm to (140.9, 88.6)
Routing:
- net LDO_ENABLE: track 16.7 -> 7.73 mm, vias 1 -> 0
- net 3V3: track 150.6 -> 152.6 mm, vias 88 -> 87
- net ATT_SER: track 34.3 -> 35.4 mm
- net Net-(IC2-RF2): track 7.47 -> 8.47 mm
- net ch1_ATT_LE: track 48.4 -> 49.0 mm
- net GND: track 0.00 -> 0.09 mm, vias 968 -> 987
- net ch1SRCLK: track 44.8 -> 44.7 mm, vias 3 -> 2
- net ch1_LNA_ON: vias 3 -> 2
- net +5V: vias 22 -> 18
Other:
- board text added: "Phase_Shifter_TestBoard"

Commit message: 色々指摘もらったので修正して発注する。
Parts:
- L1, L2, L3, L4: footprint Inductor_SMD:L_0603_1608Metric_Pad1.05x0.95mm_HandSolder -> Inductor_SMD:L_0402_1005Metric
- R13, R14: footprint Resistor_SMD:R_0603_1608Metric_Pad0.98x0.95mm_HandSolder -> Resistor_SMD:R_0402_1005Metric
- moved L4 1.62 mm to (129.1, 110.6)
- moved L3 1.47 mm to (124.6, 110.6)
- moved L2 1.36 mm to (129.4, 95.6)
- moved L1 1.26 mm to (124.6, 95.6)
- moved R13 1.17 mm to (154.0, 96.6)
- moved R14 1.13 mm to (154.0, 111.6)
- moved C11 0.62 mm to (127.7, 90.5)
- moved C12 0.44 mm to (127.8, 106.3)
Connections:
- net Net-(IC11-RF_IN) renamed /PHASE_IN_1
- net Net-(IC11-RF_OUT) renamed /ATT_IN_1
- net Net-(IC2-RF2) renamed /ATT_OUT_1
- net Net-(IC3-RF-IN) renamed /LNA_RF_IN_1
- net Net-(IC3-RF-OUT) renamed /LNA_RF_OUT_1
- net Net-(IC4-RF-IN) renamed /LNA_RF_IN_2
- net Net-(IC4-RF-OUT) renamed /LNA_RF_OUT_2
- net Net-(IC6-RF1) renamed /ATT_IN_2
- net Net-(IC6-RF2) renamed /ATT_OUT_2
- net Net-(IC9-RF_IN) renamed /PHASE_IN_2
- net Net-(J5-In) renamed /signal_1
- net Net-(J7-In) renamed /Test
- net Net-(J9-In) renamed /signal_2
Routing:
- net 3V3: track 152.6 -> 156.0 mm
- net Net-(IC3-BIASOUT): track 3.40 -> 1.53 mm
- net Net-(IC4-BIASOUT): track 3.25 -> 1.56 mm
- net ch1_SRCLR: track 40.6 -> 39.2 mm
- net /LNA_RF_OUT_2: track 4.84 -> 3.64 mm
- net /LNA_RF_IN_2: track 5.74 -> 4.67 mm
- net /LNA_RF_OUT_1: track 4.67 -> 3.74 mm
- net /LNA_RF_IN_1: track 5.61 -> 4.73 mm
- net ch1_QH: track 11.0 -> 11.9 mm
- net /ATT_OUT_1: track 8.47 -> 7.66 mm
- net ATT_SER: track 35.4 -> 36.1 mm
- net /ATT_OUT_2: track 8.40 -> 7.70 mm
- net Net-(IC9-D6): track 6.30 -> 5.76 mm
- net GND: track 0.09 -> 0.00 mm, vias 987 -> 1807
- net +5V: vias 18 -> 17
Other:
- board text added: "CH1"
- board text added: "CH2"
- board text added: "INPUT"
- board text added: "OUTPUT"
