File: MAPS-010143/MAPS-010143.kicad_sch (KiCad schematic)
At the start: 85 parts, among them IC1 LM2776DBVT, IC11 MAPS-010144-TR0500, IC2 PE4302-51, IC3 BGB_741L7ESD_E6327, IC4 BGB_741L7ESD_E6327, IC6 PE4302-51, IC7 SN74HC595NSR, IC8 SN74HC595NSR, IC9 MAPS-010144-TR0500, J13 Conn_01x02_Pin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

Commit message: v2 発注記念。
Parts:
- removed U4: TPS7A2033PDQNR, footprints:DQN0004A-MFG, symbol 2026-02-05_17-45-36:TPS7A2033PDQNR
- added IC5: TPS7A2033PDBVR, SOT95P280X145-5N, symbol SamacSys_Parts_old:TPS7A2033PDBVR
Connections:
- net +3V3: now also IC5.5 (OUT)
- net +5V: now also IC5.1 (IN)
- net GND: now also IC5.2 (GND)
- net LDO_ENABLE: now also IC5.3 (EN)

Commit message: 色々指摘もらったので修正して発注する。
Parts:
- IC5: footprint SOT95P280X145-5N -> SamacSys_Parts:SOT95P280X145-5N
- L1, L2, L3, L4: footprint Inductor_SMD:L_0603_1608Metric_Pad1.05x0.95mm_HandSolder -> Inductor_SMD:L_0402_1005Metric
- R13, R14: footprint Resistor_SMD:R_0603_1608Metric_Pad0.98x0.95mm_HandSolder -> Resistor_SMD:R_0402_1005Metric
Connections:
- net signal_2: now reaches C5.1, J9.1 (In)
- net ATT_OUT_1: now reaches IC2.14 (RF2), J6.1 (In), R13.1
- net signal_1: now reaches C3.1, J5.1 (In)
- net LNA_RF_OUT_2: now reaches C6.1, IC4.4 (RF-OUT), L4.2
- net PHASE_IN_2: now reaches C6.2, IC9.5 (RF_IN)
- net LNA_RF_OUT_1: now reaches C4.1, IC3.4 (RF-OUT), L2.2
- net PHASE_IN_1: now reaches C4.2, IC11.5 (RF_IN)
- net LNA_RF_IN_2: now reaches C5.2, IC4.3 (RF-IN), L3.2
- net LNA_RF_IN_1: now reaches C3.2, IC3.3 (RF-IN), L1.2
- net ATT_OUT_2: now reaches IC6.14 (RF2), J14.1 (In), R14.1
- net ATT_IN_1: now reaches IC11.14 (RF_OUT), IC2.2 (RF1)
- net Test: now reaches J7.1 (In), J8.1 (In)
- net ATT_IN_2: now reaches IC6.2 (RF1), IC9.14 (RF_OUT)
Other:
- moved on the sheet: C3, C5, L1, L3
Changed lines of the file:
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@@
 	)
 	(junction
-		(at 270.51 200.66)
+		(at 261.62 200.66)
 		(diameter 0)
 		(color 0 0 0 0)
@@
 	)
 	(junction
-		(at 270.51 382.27)
+		(at 260.35 382.27)
 		(diameter 0)
 		(color 0 0 0 0)
@@
 	(wire
 		(pts
-			(xy 279.4 379.73) (xy 275.59 379.73)
+			(xy 279.4 379.73) (xy 265.43 379.73)
 		)
 		(stroke
@@
 	(wire
 		(pts
-			(xy 270.51 200.66) (xy 279.4 200.66)
+			(xy 261.62 200.66) (xy 279.4 200.66)
 		)
 		(stroke
@@
 	(wire
 		(pts
-			(xy 270.51 373.38) (xy 270.51 374.65)
+			(xy 260.35 373.38) (xy 260.35 374.65)
 		)
 		(stroke
@@
 	(wire
 		(pts
-			(xy 270.51 191.77) (xy 270.51 193.04)
+			(xy 261.62 191.77) (xy 261.62 193.04)
 		)
 		(stroke
@@
 	(wire
 		(pts
-			(xy 234.95 382.27) (xy 264.16 382.27)
-		)
-		(stroke
-			(width 0)
-			(type default)
-		)
-	)
-	(wire
-		(pts
 			(xy 325.12 342.9) (xy 325.12 377.19)
 		)
@@
 	(wire
 		(pts
-			(xy 275.59 373.38) (xy 270.51 373.38)
+			(xy 265.43 373.38) (xy 260.35 373.38)
 		)
 		(stroke
@@
 	(wire
 		(pts
-			(xy 269.24 382.27) (xy 270.51 382.27)
+			(xy 259.08 382.27) (xy 260.35 382.27)
 		)
 		(stroke
@@
 	(wire
 		(pts
-			(xy 234.95 200.66) (xy 264.16 200.66)
+			(xy 234.95 200.66) (xy 255.27 200.66)
 		)
 		(stroke
@@
 	(wire
 		(pts
-			(xy 275.59 191.77) (xy 270.51 191.77)
+			(xy 275.59 191.77) (xy 261.62 191.77)
 		)
 		(stroke
@@
 	(wire
 		(pts
-			(xy 269.24 200.66) (xy 270.51 200.66)
+			(xy 260.35 200.66) (xy 261.62 200.66)
 		)
 		(stroke
@@
 	(wire
 		(pts
-			(xy 270.51 382.27) (xy 279.4 382.27)
+			(xy 260.35 382.27) (xy 279.4 382.27)
 		)
 		(stroke
@@
 	(wire
 		(pts
+			(xy 234.95 382.27) (xy 254 382.27)
+		)
+		(stroke
+			(width 0)
+			(type default)
+		)
+	)
+	(wire
+		(pts
 			(xy 368.3 78.74) (xy 368.3 77.47)
 		)
@@
 	(wire
 		(pts
-			(xy 275.59 379.73) (xy 275.59 373.38)
+			(xy 265.43 379.73) (xy 265.43 373.38)
 		)
 		(stroke
@@
 		)
 	)
+	(label "Test"
+		(at 382.27 520.7 0)
+		(effects
+			(font
+				(size 1.27 1.27)
+			)
+			(justify left bottom)
+		)
+	)
+	(label "ATT_OUT_1"
+		(at 563.88 203.2 0)
+		(effects
+			(font
+				(size 1.27 1.27)
+			)
+			(justify left bottom)
+		)
+	)
+	(label "signal_1"
+		(at 237.49 200.66 0)
+		(effects
+			(font
+				(size 1.27 1.27)
+			)
+			(justify left bottom)
+		)
+	)
+	(label "ATT_OUT_2"
+		(at 563.88 384.81 0)
+		(effects
+			(font
+				(size 1.27 1.27)
+			)
+			(justify left bottom)
+		)
+	)
+	(label "signal_2"
+		(at 240.03 382.27 0)
+		(effects
+			(font
+				(size 1.27 1.27)
+			)
+			(justify left bottom)
+		)
+	)
+	(label "LNA_RF_IN_1"
+		(at 264.16 200.66 0)
+		(effects
+			(font
+				(size 1.27 1.27)
+			)
+			(justify left bottom)
+		)
+	)
+	(label "LNA_RF_OUT_2"
+		(at 287.02 389.89 0)
+		(effects
+			(font
+				(size 1.27 1.27)
+			)
+			(justify left bottom)
+		)
+	)
+	(label "LNA_RF_OUT_1"
+		(at 284.48 208.28 0)
+		(effects
+			(font
+				(size 1.27 1.27)
+			)
+			(justify left bottom)
+		)
+	)
+	(label "ATT_IN_2"
+		(at 438.15 384.81 0)
+		(effects
+			(font
+				(size 1.27 1.27)
+			)
+			(justify left bottom)
+		)
+	)
+	(label "PHASE_IN_2"
+		(at 350.52 384.81 0)
+		(effects
+			(font
+				(size 1.27 1.27)
+			)
+			(justify left bottom)
+		)
+	)
+	(label "LNA_RF_IN_2"
+		(at 266.7 382.27 0)
+		(effects
+			(font
+				(size 1.27 1.27)
+			)
+			(justify left bottom)
+		)
+	)
+	(label "PHASE_IN_1"
+		(at 347.98 203.2 0)
+		(effects
+			(font
+				(size 1.27 1.27)
+			)
+			(justify left bottom)
+		)
+	)
+	(label "ATT_IN_1"
+		(at 449.58 203.2 0)
+		(effects
+			(font
+				(size 1.27 1.27)
+			)
+			(justify left bottom)
+		)
+	)
 	(global_label "ch2_ATT_C1"
 		(shape input)
@@
 	(symbol
 		(lib_id "Device:L")
-		(at 270.51 378.46 0)
+		(at 260.35 378.46 0)
 		(unit 1)
 		(body_style 1)
@@
 		(fields_autoplaced yes)
 		(property "Reference" "L3"
-			(at 271.7772 377.2478 0)
+			(at 261.6172 377.2478 0)
 			(show_name no)
 			(do_not_autoplace no)
@@
 		)
 		(property "Value" "22n"
-			(at 271.7772 379.6721 0)
+			(at 261.6172 379.6721 0)
 			(show_name no)
 			(do_not_autoplace no)
@@
 			)
 		)
-		(property "Footprint" "Inductor_SMD:L_0603_1608Metric_Pad1.05x0.95mm_HandSolder"
-			(at 270.51 378.46 0)
+		(property "Footprint" "Inductor_SMD:L_0402_1005Metric"
+			(at 260.35 378.46 0)
 			(hide yes)
 			(show_name no)
@@
 		)
 		(property "Datasheet" ""
-			(at 270.51 378.46 0)
+			(at 260.35 378.46 0)
 			(hide yes)
 			(show_name no)
@@
 		)
 		(property "Description" "Inductor"
-			(at 270.51 378.46 0)
+			(at 260.35 378.46 0)
 			(hide yes)
 			(show_name no)
@@
 	(symbol
 		(lib_id "Device:L")
-		(at 270.51 196.85 0)
+		(at 261.62 196.85 0)
 		(unit 1)
 		(body_style 1)
@@
 		(fields_autoplaced yes)
 		(property "Reference" "L1"
-			(at 271.7772 195.6378 0)
+			(at 262.8872 195.6378 0)
 			(show_name no)
 			(do_not_autoplace no)
@@
 		)
 		(property "Value" "22n"
-			(at 271.7772 198.0621 0)
+			(at 262.8872 198.0621 0)
 			(show_name no)
 			(do_not_autoplace no)
@@
 			)
 		)
-		(property "Footprint" "Inductor_SMD:L_0603_1608Metric_Pad1.05x0.95mm_HandSolder"
-			(at 270.51 196.85 0)
+		(property "Footprint" "Inductor_SMD:L_0402_1005Metric"
+			(at 261.62 196.85 0)
 			(hide yes)
 			(show_name no)
@@
 		)
 		(property "Datasheet" ""
-			(at 270.51 196.85 0)
+			(at 261.62 196.85 0)
 			(hide yes)
 			(show_name no)
@@
 		)
 		(property "Description" "Inductor"
-			(at 270.51 196.85 0)
+			(at 261.62 196.85 0)
 			(hide yes)
 			(show_name no)
@@
 			)
 		)
-		(property "Footprint" "Resistor_SMD:R_0603_1608Metric_Pad0.98x0.95mm_HandSolder"
+		(property "Footprint" "Resistor_SMD:R_0402_1005Metric"
 			(at 582.93 387.35 0)
 			(hide yes)
@@
 			)
 		)
-		(property "Footprint" "Inductor_SMD:L_0603_1608Metric_Pad1.05x0.95mm_HandSolder"
+		(property "Footprint" "Inductor_SMD:L_0402_1005Metric"
 			(at 335.28 377.19 0)
 			(hide yes)
@@
 	(symbol
 		(lib_id "Device:C_Small")
-		(at 266.7 382.27 90)
+		(at 256.54 382.27 90)
 		(unit 1)
 		(body_style 1)
@@
 		(fields_autoplaced yes)
 		(property "Reference" "C5"
-			(at 266.7063 376.5634 90)
+			(at 256.5463 376.5634 90)
 			(show_name no)
 			(do_not_autoplace no)
@@
 		)
 		(property "Value" "33p"
-			(at 266.7063 378.9877 90)
+			(at 256.5463 378.9877 90)
 			(show_name no)
 			(do_not_autoplace no)
@@
 		)
 		(property "Footprint" "Capacitor_SMD:C_0402_1005Metric_Pad0.74x0.62mm_HandSolder"
-			(at 266.7 382.27 0)
+			(at 256.54 382.27 0)
 			(hide yes)
 			(show_name no)
@@
 		)
 		(property "Datasheet" ""
-			(at 266.7 382.27 0)
+			(at 256.54 382.27 0)
 			(hide yes)
 			(show_name no)
@@
 		)
 		(property "Description" "Unpolarized capacitor, small symbol"
-			(at 266.7 382.27 0)
+			(at 256.54 382.27 0)
 			(hide yes)
 			(show_name no)
@@
 	(symbol
 		(lib_id "Device:C_Small")
-		(at 266.7 200.66 90)
+		(at 257.81 200.66 90)
 		(unit 1)
 		(body_style 1)
@@
 		(fields_autoplaced yes)
 		(property "Reference" "C3"
-			(at 266.7063 194.9534 90)
+			(at 257.8163 194.9534 90)
 			(show_name no)
 			(do_not_autoplace no)
@@
 		)
 		(property "Value" "33p"
-			(at 266.7063 197.3777 90)
+			(at 257.8163 197.3777 90)
 			(show_name no)
 			(do_not_autoplace no)
@@
 		)
 		(property "Footprint" "Capacitor_SMD:C_0402_1005Metric_Pad0.74x0.62mm_HandSolder"
-			(at 266.7 200.66 0)
+			(at 257.81 200.66 0)
 			(hide yes)
 			(show_name no)
@@
 		)
 		(property "Datasheet" ""
-			(at 266.7 200.66 0)
+			(at 257.81 200.66 0)
 			(hide yes)
 			(show_name no)
@@
 		)
 		(property "Description" "Unpolarized capacitor, small symbol"
-			(at 266.7 200.66 0)
+			(at 257.81 200.66 0)
 			(hide yes)
 			(show_name no)
@@
 			)
 		)
-		(property "Footprint" "Inductor_SMD:L_0603_1608Metric_Pad1.05x0.95mm_HandSolder"
+		(property "Footprint" "Inductor_SMD:L_0402_1005Metric"
 			(at 335.28 195.58 0)
 			(hide yes)
@@
 			)
 		)
-		(property "Footprint" "SOT95P280X145-5N"
+		(property "Footprint" "SamacSys_Parts:SOT95P280X145-5N"
 			(at 356.87 39.37 0)
 			(hide yes)
@@
 			)
 		)
-		(property "Footprint" "Resistor_SMD:R_0603_1608Metric_Pad0.98x0.95mm_HandSolder"
+		(property "Footprint" "Resistor_SMD:R_0402_1005Metric"
 			(at 582.93 205.74 0)
 			(hide yes)
